Commit message: 2 robot sim add

File: p2os_urdf/defs/pioneer3dx_body.xacro (robot description, xacro)
@@ -3,8 +3,8 @@
   <xacro:include filename="$(find p2os_urdf)/defs/pioneer3dx_wheel.xacro"/>
   <!-- Chassis description -->
-  <link name="base_link">
+  <link name="$(arg ns)/base_link">
 	<!-- CHECK THESE VALUES. THEY MAY BE COMPLETELY WRONG. -->
 	<inertial>
-	  <mass value="20.0"/>
+	  <mass value="13.0"/>
 	  <origin xyz="-0.045 0 0.148"/>
 	  <inertia ixx="0.3338" ixy="0.0" ixz="0.0"
@@ -31,8 +31,8 @@
 	</collision>
   </link>
-  <gazebo reference="base_link">
+  <gazebo reference="$(arg ns)/base_link">
 	<material value="Gazebo/Red"/>
   </gazebo>
-  <link name="top_plate">
+  <link name="$(arg ns)/top_plate">
 	<inertial>
 	  <mass value="0.01"/>
@@ -52,14 +52,14 @@
 	</visual>
   </link>
-  <gazebo reference="top_plate">
-	<material value="Gazebo/Black"/>
-  </gazebo>
-  <joint name="base_top_joint" type="fixed">
+  <gazebo reference="$(arg ns)/top_plate">
+	<material value="Gazebo/Black"/>
+  </gazebo>
+  <joint name="$(arg ns)/base_top_joint" type="fixed">
 	<origin xyz="-0.045 0 0.24" rpy="0 0 0"/>
-	<parent link="base_link"/>
-	<child link="top_plate"/>
+	<parent link="$(arg ns)/base_link"/>
+	<child link="$(arg ns)/top_plate"/>
   </joint>
   <!-- Swivel -->
-  <link name="swivel">
+  <link name="$(arg ns)/swivel">
 	<inertial>
 	  <mass value="0.1"/>
@@ -78,17 +78,17 @@
 	</visual>
   </link>
-  <gazebo reference="swivel">
-	<material value="Gazebo/Black"/>
-  </gazebo>
-  <joint name="base_swivel_joint" type="continuous">
+  <gazebo reference="$(arg ns)/swivel">
+	<material value="Gazebo/Black"/>
+  </gazebo>
+  <joint name="$(arg ns)/base_swivel_joint" type="continuous">
 	<origin xyz="-0.185 0 0.055" rpy="0 0 0"/>
 	<axis xyz="0 0 1"/>
     <limit effort="100" velocity="100" k_velocity="0" />
     <joint_properties damping="0.0" friction="0.0" />
-	<parent link="base_link"/>
-	<child link="swivel"/>
+	<parent link="$(arg ns)/base_link"/>
+	<child link="$(arg ns)/swivel"/>
   </joint>
   <!-- Center Wheel + Hubcap -->
-  <link name="center_hubcap">
+  <link name="$(arg ns)/center_hubcap">
     <inertial>
 	  <mass value="0.01"/>
@@ -107,8 +107,8 @@
 	</visual>
   </link>
-  <gazebo reference="center_hubcap">
-	<material value="Gazebo/Black"/>
-  </gazebo>
-  <joint name="swivel_hubcap_joint" type="continuous">
+  <gazebo reference="$(arg ns)/center_hubcap">
+	<material value="Gazebo/Black"/>
+  </gazebo>
+  <joint name="$(arg ns)/swivel_hubcap_joint" type="continuous">
 	<origin xyz="-0.026 0 -0.016" rpy="0 0 0"/>
 	<axis xyz="0 1 0"/>
@@ -116,8 +116,8 @@
     <limit effort="100" velocity="100" k_velocity="0" />
     <joint_properties damping="0.0" friction="0.0" />
-	<parent link="swivel"/>
-	<child link="center_wheel"/>
-  </joint>
-  <link name="center_wheel">
+	<parent link="$(arg ns)/swivel"/>
+	<child link="$(arg ns)/center_wheel"/>
+  </joint>
+  <link name="$(arg ns)/center_wheel">
 	<inertial>
 	  <mass value="0.1"/>
@@ -143,16 +143,16 @@
 	</collision>
   </link>
-  <gazebo reference="center_wheel">
-	<material value="Gazebo/Black"/>
-  </gazebo>
-  <joint name="center_wheel_joint" type="fixed">
+  <gazebo reference="$(arg ns)/center_wheel">
+	<material value="Gazebo/Black"/>
+  </gazebo>
+  <joint name="$(arg ns)/center_wheel_joint" type="fixed">
 	<origin xyz="-0.0035 0 -0.001" rpy="0 0 0"/>
-	<parent link="center_wheel"/>
-	<child link="center_hubcap"/>
-  </joint>
-  <xacro:p3dx_wheel suffix="left" parent="base_link" reflect="1"/>
-  <xacro:p3dx_wheel suffix="right" parent="base_link" reflect="-1"/>
+	<parent link="$(arg ns)/center_wheel"/>
+	<child link="$(arg ns)/center_hubcap"/>
+  </joint>
+  <xacro:p3dx_wheel suffix="left" parent="$(arg ns)/base_link" reflect="1" namespace="$(arg ns)"/>
+  <xacro:p3dx_wheel suffix="right" parent="$(arg ns)/base_link" reflect="-1" namespace="$(arg ns)"/>
   <!-- Front + Back Sonar -->
-  <link name="front_sonar">
+  <link name="$(arg ns)/front_sonar">
 	<inertial>
 	  <mass value="0.0001"/>
@@ -171,13 +171,13 @@
 	</visual>
   </link>
-  <gazebo reference="front_sonar">
+  <gazebo reference="$(arg ns)/front_sonar">
 	<material value="Gazebo/Yellow"/>
   </gazebo>
-  <joint name="base_front_joint" type="fixed">
+  <joint name="$(arg ns)/base_front_joint" type="fixed">
 	<origin xyz="-0.198 0 0.208" rpy="0 0 0"/>
-	<parent link="base_link"/>
-	<child link="front_sonar"/>
-  </joint>
-  <link name="back_sonar">
+	<parent link="$(arg ns)/base_link"/>
+	<child link="$(arg ns)/front_sonar"/>
+  </joint>
+  <link name="$(arg ns)/back_sonar">
 	<inertial>
 	  <mass value="0.0001"/>
@@ -196,31 +196,31 @@
 	</visual>
   </link>
-  <gazebo reference="back_sonar">
+  <gazebo reference="$(arg ns)/back_sonar">
 	<material value="Gazebo/Yellow"/>
   </gazebo>
-  <joint name="base_back_joint" type="fixed">
+  <joint name="$(arg ns)/base_back_joint" type="fixed">
 	<origin xyz="0.109 0 0.209" rpy="0 0 0"/>
 	<!-- <origin xyz="0 0 0" rpy="0 0 0"/> -->
-	<parent link="base_link"/>
-	<child link="back_sonar"/>
+	<parent link="$(arg ns)/base_link"/>
+	<child link="$(arg ns)/back_sonar"/>
   </joint>
   <gazebo>
     <!-- Robot locomotion plugin -->
-	<plugin name="differential_drive_controller" filename="libgazebo_ros_diff_drive.so">
+	<plugin name="$(arg ns)/differential_drive_controller" filename="libgazebo_ros_diff_drive.so">
       <legacyMode>false</legacyMode>
       <alwaysOn>true</alwaysOn>
 	  <updateRate>100.0</updateRate>
-	  <leftJoint>base_left_wheel_joint</leftJoint>
-      <rightJoint>base_right_wheel_joint</rightJoint>
+	  <leftJoint>$(arg ns)/base_left_wheel_joint</leftJoint>
+      <rightJoint>$(arg ns)/base_right_wheel_joint</rightJoint>
 	  <wheelSeparation>0.32</wheelSeparation>
 	  <wheelDiameter>0.18</wheelDiameter>
 	  <wheelTorque>5</wheelTorque>
       <wheelAcceleration>0</wheelAcceleration>
-      <robotNamespace>pioneer</robotNamespace>
-	  <commandTopic>cmd_vel</commandTopic>
-	  <odometryTopic>odom</odometryTopic>
+      <!--<robotNamespace>$(arg ns)</robotNamespace>-->
+	  <commandTopic>$(arg ns)/cmd_vel</commandTopic>
+	  <odometryTopic>$(arg ns)/odom</odometryTopic>
       <odometrySource>ENCODER</odometrySource><!--Other option is World-->
-	  <odometryFrame>odom</odometryFrame>
-      <robotBaseFrame>base_link</robotBaseFrame>
+	  <odometryFrame>$(arg ns)/odom</odometryFrame>
+      <robotBaseFrame>$(arg ns)/base_link</robotBaseFrame>
       <publishTf>1</publishTf>
       <publishWheelTF>false</publishWheelTF>
@@ -229,9 +229,9 @@
 	</plugin>
     <!-- Fake localization plugin -->
-    <plugin name="ground_truth_odometry" filename="libgazebo_ros_p3d.so">
+    <plugin name="$(arg ns)/ground_truth_odometry" filename="libgazebo_ros_p3d.so">
 	  <alwaysOn>true</alwaysOn>
 	  <updateRate>100.0</updateRate>
-	  <bodyName>base_link</bodyName>
-	  <topicName>base_pose_ground_truth</topicName>
+	  <bodyName>$(arg ns)/base_link</bodyName>
+	  <topicName>$base_pose_ground_truth</topicName>
 	  <gaussianNoise>0.01</gaussianNoise>
 	  <frameName>map</frameName>-->
@@ -239,4 +239,5 @@
 	  <xyzOffsets>0 0 0</xyzOffsets>
 	  <rpyOffsets>0 0 0</rpyOffsets>
+	  <robotNamespace>$(arg ns)</robotNamespace>
 	</plugin>
   </gazebo>

File: p2os_urdf/defs/pioneer3dx_wheel.xacro (robot description, xacro)
@@ -5,6 +5,6 @@
   <xacro:property name="M_PI" value="3.14159"/>
   <!-- Right/Left Hubcap + Wheel -->
-  <xacro:macro name="p3dx_wheel" params="suffix parent reflect">
-    <link name="p3dx_${suffix}_wheel">
+  <xacro:macro name="p3dx_wheel" params="suffix parent reflect namespace">
+    <link name="${namespace}/p3dx_${suffix}_wheel">
       <inertial>
         <mass value="0.5"/>
@@ -29,10 +29,10 @@
       </collision>
     </link>
-    <joint name="base_${suffix}_hubcap_joint" type="fixed">
+    <joint name="${namespace}/base_${suffix}_hubcap_joint" type="fixed">
       <origin xyz="0 0 0" rpy="0 0 0"/>
-      <parent link="p3dx_${suffix}_wheel"/>
-      <child link="p3dx_${suffix}_hubcap"/>
+      <parent link="${namespace}/p3dx_${suffix}_wheel"/>
+      <child link="${namespace}/p3dx_${suffix}_hubcap"/>
     </joint>
-    <link name="p3dx_${suffix}_hubcap">
+    <link name="${namespace}/p3dx_${suffix}_hubcap">
       <inertial>
         <mass value="0.01"/>
@@ -57,5 +57,5 @@
         <mechanicalReduction>${reflect * 624/35 * 80/19}</mechanicalReduction>
         </transmission>-->
-    <joint name="base_${suffix}_wheel_joint" type="continuous">
+    <joint name="${namespace}/base_${suffix}_wheel_joint" type="continuous">
       <axis xyz="0 1 0"/>
       <anchor xyz="0 0 0"/>
@@ -63,11 +63,11 @@
       <joint_properties damping="0.0" friction="0.0" />
       <origin xyz="0 ${reflect*0.158} 0.091" rpy="0 0 0"/>
-      <parent link="base_link"/>
-      <child link="p3dx_${suffix}_wheel"/>
+      <parent link="${parent}"/>
+      <child link="${namespace}/p3dx_${suffix}_wheel"/>
     </joint>
-    <gazebo reference="p3dx_${suffix}_hubcap">
+    <gazebo reference="${namespace}/p3dx_${suffix}_hubcap">
       <material value="Gazebo/Yellow"/>
     </gazebo>
-    <gazebo reference="p3dx_${suffix}_wheel">
+    <gazebo reference="${namespace}/p3dx_${suffix}_wheel">
       <material value="Gazebo/Black"/>
       <mu1>0.5</mu1>

Commit message: add lift platform

File: p2os_urdf/defs/pioneer3dx_body.xacro (robot description, xacro)
@@ -2,4 +2,5 @@
 <robot xmlns:xacro="http://ros.org/wiki/xacro">
   <xacro:include filename="$(find p2os_urdf)/defs/pioneer3dx_wheel.xacro"/>
+  <xacro:include filename="$(find p2os_urdf)/defs/inertia_calculation.xacro"/>
   <!-- Chassis description -->
   <link name="$(arg ns)/base_link">
@@ -205,4 +206,51 @@
 	<child link="$(arg ns)/back_sonar"/>
   </joint>
+  <joint name="$(arg ns)/lift_joint" type="prismatic">
+        <origin xyz="-0.05 0 0.3" rpy="0 0 0"/>
+        <parent link="$(arg ns)/base_link"/>
+        <child link="$(arg ns)/lift"/>
+        <axis xyz="0 0 1"/>
+        <limit lower="0" upper="0.5" velocity="0.5" effort="100"/>
+    </joint>
+  <link name="$(arg ns)/lift">
+        <visual>
+            <origin xyz="0 0 -0.001" rpy="0 0 0"/>
+            <geometry>
+                <box size="0.2 0.2 0.02" />
+            </geometry>
+            <material name="SonarYellow">
+				<color rgba="0.715 0.583 0.210 1.0"/>
+	  		</material>
+        </visual>
+        <collision>
+            <origin xyz="0 0 -0.001" rpy="0 0 0"/>
+            <geometry>
+                <box size="0.2 0.2 0.02" />
+            </geometry>
+        </collision>
+        <xacro:inertial_box mass="0.5" x="0.2" y="0.2" z="0.02">
+            <origin xyz="0 0 -0.001" rpy="0 0 0"/>
+        </xacro:inertial_box>
+    </link>
+    <gazebo reference="$(arg ns)/lift">
+		<material value="Gazebo/Orange"/>
+		<mu1 value="100"/>
+		<mu2 value="100"/>
+  	</gazebo>
+  	<gazebo>
+  		<plugin name="gazebo_ros_control" filename="libgazebo_ros_control.so">
+			<robotNamespace>$(arg ns)</robotNamespace>
+	  	</plugin>
+	</gazebo>
+	<transmission name="$(arg ns)/lift_transmission">
+    <type>transmission_interface/SimpleTransmission</type>
+    <joint name="$(arg ns)/lift_joint">
+      <hardwareInterface>hardware_interface/EffortJointInterface</hardwareInterface>
+    </joint>
+    <actuator name="$(arg ns)/motor1">
+      <hardwareInterface>hardware_interface/EffortJointInterface</hardwareInterface>
+      <mechanicalReduction>1</mechanicalReduction>
+    </actuator>
+  </transmission>
   <gazebo>
     <!-- Robot locomotion plugin -->

Commit message: Platform height change

File: p2os_urdf/defs/pioneer3dx_body.xacro (robot description, xacro)
@@ -207,5 +207,5 @@
   </joint>
   <joint name="$(arg ns)/lift_joint" type="prismatic">
-        <origin xyz="-0.05 0 0.3" rpy="0 0 0"/>
+        <origin xyz="-0.05 0 0.35" rpy="0 0 0"/>
         <parent link="$(arg ns)/base_link"/>
         <child link="$(arg ns)/lift"/>
